File: sch/main.sch (EAGLE design)
At the start: 37 parts

Commit message: [ update ] schematics version, silkscreen
Other:
- note added: "ooklone_v001"
- note removed: "ooklone_v000"
Changed lines of the file:
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@@
 <text x="-15.24" y="-43.18" size="1.778" layer="97">connect to common</text>
 <text x="78.74" y="-43.18" size="1.778" layer="97">connect to common</text>
-<text x="53.34" y="-63.5" size="1.778" layer="94" font="vector">ooklone_v000</text>
+<text x="53.34" y="-63.5" size="1.778" layer="94" font="vector">ooklone_v001</text>
 <text x="53.34" y="-68.58" size="1.778" layer="94" font="vector">https://github.com/texane/ooklone</text>
 <text x="53.34" y="-73.66" size="1.778" layer="94" font="vector">texane@gmail.com</text>
